Commit message: kinda webserver dummy zwischenstand

File: catkin_ws/src/nexus_4wd_mecanum_simulator/nexus_4wd_mecanum_description/urdf/nexus_4wd_mecanum.xacro (robot description, xacro)
@@ -328,5 +328,5 @@
   <xacro:include filename="$(find realsense_gazebo_plugin)/urdf/_d435.urdf.xacro" />
     <xacro:sensor_d435 parent="base_link">
-      <origin xyz="0.20 0 0.05" rpy="0 0.20 0"/>
+      <origin xyz="0.20 0 0.10" rpy="0 0.05 0"/>
   </xacro:sensor_d435>
   <!-- Include controller plugin for Gazebo -->
@@ -343,4 +343,5 @@
   <xacro:urm04_sensor frame_name="rear_sensor" ros_topic="rear_sensor" update_rate="10" min_range="0.04" max_range="2.5" horizontal_field_of_view="1.04" vertical_field_of_view="0.04" ray_count="2" />
   <!-- Lidar -->
+  <!--
   <joint name="lidar_joint" type="fixed">
     <origin xyz="0.0 0.0 0.30" rpy="0 0 0" />
@@ -383,3 +384,4 @@
     </sensor>
   </gazebo>
+  -->
 </robot>

File: catkin_ws/src/nexus_4wd_mecanum_simulator/realsense_gazebo_plugin/urdf/_d435.gazebo.xacro (robot description, xacro)
@@ -27,6 +27,6 @@
           <horizontal_fov>${69.4*deg_to_rad}</horizontal_fov>
           <image>
-            <width>960</width> <!-- 1920 -->
-            <height>540</height> <!-- 1080 -->
+            <width>1920</width> <!-- 1920 -->
+            <height>1080</height> <!-- 1080 -->
             <format>RGB_INT8</format>
           </image>
